File: Charger.sch (EAGLE design)
At the start: 14 parts, among them Q1 SPP80P06P

Commit message: Finished BRD
Parts:
- LED1: device led:LED5MM -> led:LEDCHIPLED_1206
Changed lines of the file:
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@@
 <setting verticaltext="up"/>
 </settings>
-<grid distance="0.1" unitdist="inch" unit="inch" style="lines" multiple="1" display="yes" altdistance="0.01" altunitdist="inch" altunit="inch"/>
+<grid distance="0.1" unitdist="inch" unit="inch" style="lines" multiple="1" display="no" altdistance="0.01" altunitdist="inch" altunit="inch"/>
 <layers>
 <layer number="1" name="Top" color="4" fill="1" visible="no" active="no"/>
@@
 <part name="R1" library="resistor" deviceset="R-EU_" device="R0805" value="0.22"/>
 <part name="R2" library="resistor" deviceset="R-EU_" device="R0805" value="100k"/>
-<part name="LED1" library="led" deviceset="LED" device="5MM"/>
+<part name="LED1" library="led" deviceset="LED" device="CHIPLED_1206"/>
 <part name="Q1" library="transistor-fet" deviceset="SPP80P06P" device=""/>
 <part name="C1" library="resistor" deviceset="CPOL-US" device="153CLV-0505"/>
